File: RGBtlc.sch (EAGLE design)
At the start: 18 parts, among them U1 TLC5940-NT

Commit message: V2, now with daisy chain ports
Parts:
- added BLANK., GND., GSCLK., SCLK., VCC., XLAT.: (no value), pinhead:PINHD-1X1
- U$1, U$2, U$3, U$4, U$5: device SparkFun-LED:LED_PIRANHA_5MM -> jim:LED_PIRANHA_5MM
Connections:
- removed net N$10: U$3.RED, U1.OUT7
- new net N$23: U$3.RED, U1.OUT8
- net GND: now also GND..1
- net N$12: now also U$2.RED; no longer U$2.BLU
- net N$13: now also U$2.BLU; no longer U$2.RED
- net N$15: now also U$1.RED; no longer U$1.BLU
- net N$16: now also U$1.BLU; no longer U$1.RED
- net N$17: now also SCLK..1
- net N$19: now also XLAT..1
- net N$2: now also U$5.RED; no longer U$5.BLU
- net N$20: now also GSCLK..1
- net N$3: now also U$5.BLU; no longer U$5.RED
- net N$4: now also U1.OUT7; no longer U1.OUT8
- net N$6: now also U$4.RED; no longer U$4.BLU
- net N$7: now also U$4.BLU; no longer U$4.RED
- net N$9: now also BLANK..1; no longer R2.1
- net VCC: now also U$1.A, U$2.A, U$3.A, U$4.A, U$5.A, VCC..1; no longer R2.2, U$1.C, U$2.C, U$3.C, U$4.C, U$5.C
Other:
- moved on the sheet: R2
